File: examples/mcu-board/mcu-board.kicad_pcb (KiCad board)
At the start: 2 copper layers, 80 x 50 mm, 15 parts, among them J1 5V_IN, J2 PROG/IO, SW1 Reset, U1 MCU, U2 AMS1117-3.3

Commit message: demo: mcu-board temp sensor + routing rework
Demo diff for the kicadiff PR-triggered workflow. Adds a temperature
sensor IC near the MCU, reworks tracking around the LDO, and wiggles
silkscreen labels — gives the visual diff something to chew on with
all three categories (add / delete / change) present.

Not a real design change. Branch exists to exercise the kicad-pr-diff
workflow against a real PR context.

Co-Authored-By: Claude Opus 4.7 (1M context) <noreply@anthropic.com>
Parts:
- added C4: 100nF, C_0805_2012Metric, F.Cu at (115.0, 132.0)
- added U3: MCP9700A, SOT-23, F.Cu at (110.0, 132.0)
Connections:
- D1 pad 1: GND -> Net-(D1-A)
- R2 pad 2: GND -> Net-(D1-A)
Routing:
- net +3V3: track 32.2 -> 102.7 mm, vias 0 -> 2
- net /PA3: track 35.0 -> 70.7 mm
- net GND: track 10.1 -> 17.9 mm, vias 2 -> 9
- net Net-(D1-A): track 0.00 -> 6.15 mm
- net /PA1: track 38.4 -> 41.5 mm, vias 2 -> 1
- net /PA2: track 38.9 -> 42.0 mm, vias 2 -> 1
- net /RST: track 82.9 -> 80.5 mm, vias 0 -> 2
- net /LED_A: track 11.0 -> 12.0 mm
